File: hardware/kicad/pico_bmc.kicad_pcb (KiCad board)
At the start: 2 copper layers, 38.1 x 52.7 mm, 7 parts, among them J1 PW_STATE, J2 PW_SWITCH, Q1 NMOS, Q2 PMOS, U1 RaspberryPi_Pico_W_SecondaryP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

Commit message: initial hardware design
Parts:
- removed J1: PW_STATE, Connector_PinHeader_2.00mm:PinHeader_1x02_P2.00mm_Vertical
- removed J2: PW_SWITCH, Connector_PinHeader_2.00mm:PinHeader_1x02_P2.00mm_Vertical
- removed Q1: NMOS, Package_TO_SOT_SMD:SOT-23
- removed Q2: PMOS, Package_TO_SOT_SMD:SOT-23
- removed R1, R2: 1k, Resistor_SMD:R_0805_2012Metric
- removed U1: RaspberryPi_Pico_W_SecondaryPins, Module_RaspberryPi_Pico:RaspberryPi_Pico_W_SMD
Routing:
- net GND: track 112.8 -> 0.00 mm
- net PW_SWITCH_SIG: track 16.9 -> 0.00 mm
- net PW_STATE_SIG: track 16.9 -> 0.00 mm
- net Net-(J2-Pin_1): track 7.38 -> 0.00 mm
- net Net-(J1-Pin_1): track 6.77 -> 0.00 mm
- net Net-(Q2-G): track 3.82 -> 0.00 mm
- net Net-(Q1-D): track 3.59 -> 0.00 mm
- net unconnected-(U1-GPIO1-Pad2): track 1.59 -> 0.00 mm
- net unconnected-(U1-GPIO0-Pad1): track 0.67 -> 0.00 mm
- removed copper zone on B.Cu, net GND
Other:
- board outline removed
- copper layers 2 -> 4
