File: hardware/kicad/pico_bmc.kicad_sch (KiCad schematic)
At the start: 7 parts, among them J1 PW_STATE, J2 PW_SWITCH, Q1 NMOS, Q2 PMOS, U1 RaspberryPi_Pico_W_SecondaryP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

Commit message: initial hardware design
Parts:
- removed J2: PW_SWITCH, Connector_PinHeader_2.00mm:PinHeader_1x02_P2.00mm_Vertical, symbol Connector:Conn_01x02_Pin
- removed Q2: PMOS, Package_TO_SOT_SMD:SOT-23, symbol Simulation_SPICE:PMOS
- added C1, C12, C13, C14, C15, C18, C19, C2, C20, C22, C23, C24, C3, C4, C6, C7, C8, C9: 0.1u, Capacitor_SMD:C_0402_1005Metric, symbol Device:C
- added C10, C11, C16, C5: 10u, Capacitor_SMD:C_0603_1608Metric, symbol Device:C
- added C17: 4.7u, Capacitor_SMD:C_0603_1608Metric, symbol Device:C
- added FB1, FB2, FB3, FB4: BLM18RK601SN1D, Inductor_SMD:L_0603_1608Metric, symbol Device:FerriteBead
- added J3: HDMI_A, Connector_Video:HDMI_A_Molex_208658-1001_Horizontal, symbol Connector:HDMI_A
- added J4: PW_STATE_OUT, Connector_PinHeader_2.00mm:PinHeader_1x02_P2.00mm_Vertical, symbol Connector:Conn_01x02_Pin
- added J5: PW_SWITCH_IN, Connector_PinHeader_2.00mm:PinHeader_1x02_P2.00mm_Vertical, symbol Connector:Conn_01x02_Pin
- added J6: PW_SWITCH_OUT, Connector_PinHeader_2.00mm:PinHeader_1x02_P2.00mm_Vertical, symbol Connector:Conn_01x02_Pin
- added P1: USB_C_Plug, symbol Connector:USB_C_Plug
- added Q2: NMOS, Package_TO_SOT_SMD:SOT-23, symbol Simulation_SPICE:NMOS
- added R3, R4: 2.2k, Resistor_SMD:R_0402_1005Metric, symbol Device:R
- added R5, R6: 4.7k, Resistor_SMD:R_0402_1005Metric, symbol Device:R
- added R7: 5.1k, symbol Device:R
- added U2: TFP401APZPR, Package_QFP:TQFP-100-1EP_14x14mm_P0.5mm_EP5x5mm_ThermalVias, symbol 2024-08-11_03-25-27:TFP401APZPR
- added U3: TXS0102DCT, Package_SO:SSOP-8_2.95x2.8mm_P0.65mm, symbol Logic_LevelTranslator:TXS0102DCT
- J1: value PW_STATE -> PW_STATE_IN
Connections:
- net GND: now also C1.1, C10.2, C11.2, C12.2, C13.2, C14.2, C15.2, C16.2, C17.2, C18.2, C19.2, C2.1, C20.2, C22.2, C23.2, C24.2, C3.2, C4.2, C5.2, C6.2, C7.2, C8.2, C9.2, J3.11 (CKS), J3.17 (GND), J3.2 (D2S), J3.5 (D1S), J3.8 (D0S), J3.SH, J4.2 (Pin_2), J5.2 (Pin_2), J6.2 (Pin_2), P1.A1 (GND), P1.A12 (GND), P1.B1 (GND), P1.B12 (GND), P1.S1 (SHIELD), Q2.3 (S), R7.2, U2.1 (DFO), U2.100 (OCK_INV), U2.101 (EPAD), U2.19 (OGND), U2.28 (OGND), U2.3 (ST), U2.39 (GND), U2.4 (PIXS), U2.45 (OGND), U2.5 (GND), U2.58 (OGND), U2.68 (GND), U2.7 (*STAG), U2.76 (OGND), U2.79 (AGND), U2.83 (AGND), U2.87 (AGND), U2.89 (AGND), U2.92 (AGND), U2.97 (PVDD), U2.98 (PGND), U3.2 (GND)
- net PW_STATE_SIG: now also U1.27 (GPIO21); no longer U1.12 (GPIO9)
- net PICO_IN_VID_SCA: now reaches U1.1 (GPIO0)
- net PICO_IN_VID_SCA: now also R5.2, U3.4 (A2)
- net TFP401_G2: now reaches U1.10 (GPIO7)
- net TFP401_G2: now also U2.22 (QE10)
- net TFP401_G3: now reaches U1.11 (GPIO8)
- net TFP401_G3: now also U2.23 (QE11)
- net TFP401_G5: now reaches U1.14 (GPIO10)
- net TFP401_G5: now also U2.25 (QE13)
- net TFP401_G6: now reaches U1.15 (GPIO11)
- net TFP401_G6: now also U2.26 (QE14)
- net TFP401_G7: now reaches U1.16 (GPIO12)
- net TFP401_G7: now also U2.27 (QE15)
- net TFP401_B3: now reaches U1.17 (GPIO13)
- net TFP401_B3: now also U2.13 (QE3)
- net TFP401_B4: now reaches U1.19 (GPIO14)
- net TFP401_B4: now also U2.14 (QE4)
- net PICO_IN_VID_SCL: now reaches U1.2 (GPIO1)
- net PICO_IN_VID_SCL: now also R6.2, U3.5 (A1)
- net TFP401_B5: now reaches U1.20 (GPIO15)
- net TFP401_B5: now also U2.15 (QE5)
- net TFP401_B6: now reaches U1.21 (GPIO16)
- net TFP401_B6: now also U2.16 (QE6)
- net TFP401_B7: now reaches U1.22 (GPIO17)
- net TFP401_B7: now also U2.17 (QE7)
- net USB_D-: now reaches U1.24 (GPIO18)
- net USB_D-: now also P1.A7 (D-)
- net USB_D+: now reaches U1.25 (GPIO19)
- net USB_D+: now also P1.A6 (D+)
- net VID_IN_HPD: now reaches U1.26 (GPIO20)
- net VID_IN_HPD: now also J3.19 (HPD)
- net TFP401_HSYNC: now reaches U1.31 (GPIO26_ADC0)
- net TFP401_HSYNC: now also U2.48 (HSYNC)
- net TFP401_VSYNC: now reaches U1.32 (GPIO27_ADC1)
- net TFP401_VSYNC: now also U2.47 (VSYNC)
- net TFP401_DE: now reaches U1.34 (GPIO28_ADC2)
- net TFP401_DE: now also U2.46 (DE)
- net PICO_3V3: now reaches U1.36 (3V3)
- net PICO_3V3: now also C1.2, R5.1, R6.1, U3.3 (VCCA), U3.6 (OE)
- net TFP401_R3: now reaches U1.4 (GPIO2)
- net TFP401_R3: now also U2.33 (QE19)
- net +5V: now reaches U1.40 (VBUS)
- net +5V: now also P1.A4 (VBUS), P1.A9 (VBUS), P1.B4 (VBUS), P1.B9 (VBUS)
- net TFP401_R4: now reaches U1.5 (GPIO3)
- net TFP401_R4: now also U2.34 (QE20)
- net TFP401_R5: now reaches U1.6 (GPIO4)
- net TFP401_R5: now also U2.35 (QE21)
- net TFP401_R6: now reaches U1.7 (GPIO5)
- net TFP401_R6: now also U2.36 (QE22)
- net TFP401_R7: now reaches U1.9 (GPIO6)
- net TFP401_R7: now also U2.37 (QE23)
- net at J1.1 (Pin_1), Q1.2 (G): now also J4.1 (Pin_1)
- net at R2.1: now also Q2.2 (G)
- new net: J5.1 (Pin_1), J6.1 (Pin_1), Q2.1 (D)
- new net: P1.A5 (CC), R7.1
- new net +3V3: FB1.2, FB2.2, FB3.2, FB4.2, U2.99 (RSVD)
- new net HDMI_5V: C2.2, J3.18 (+5V), R3.1, R4.1, U3.7 (VCCB)
- new net TFP401_AVDD: C5.1, C6.1, C7.1, C8.1, C9.1, FB2.1, U2.82 (AVDD), U2.84 (AVDD), U2.88 (AVDD), U2.95 (AVDD)
- new net TFP401_CAP: C17.1, C22.1
- new net TFP401_DVDD: C10.1, C23.1, C3.1, C4.1, FB1.1, U2.38 (DVDD), U2.6 (DVDD), U2.67 (DVDD)
- new net TFP401_G4: U1.12 (GPIO9), U2.24 (QE12)
- new net TFP401_OVDD: C11.1, C12.1, C13.1, C14.1, C15.1, C24.1, FB3.1, U2.18 (OVDD), U2.29 (OVDD), U2.43 (OVDD), U2.57 (OVDD), U2.78 (OVDD)
- new net TFP401_PVDD: C16.1, C18.1, C19.1, C20.1, FB4.1
- new net VID_IN_CLK+: J3.10 (CK+), U2.93 (RXC+)
- new net VID_IN_CLK-: J3.12 (CK-), U2.94 (RXC-)
- new net VID_IN_D0+: J3.7 (D0+), U2.90 (RX0+)
- new net VID_IN_D0-: J3.9 (D0-), U2.91 (RX0-)
- new net VID_IN_D1+: J3.4 (D1+), U2.85 (RX1+)
- new net VID_IN_D1-: J3.6 (D1-), U2.86 (RX1-)
- new net VID_IN_D2+: J3.1 (D2+), U2.80 (RX2+)
- new net VID_IN_D2-: J3.3 (D2-), U2.81 (RX2-)
- new net VID_IN_SCL: J3.15 (SCL), R4.2, U3.8 (B1)
- new net VID_IN_SDA: J3.16 (SDA), R3.2, U3.1 (B2)
- no-connect marks 38 -> 65
Other:
- moved on the sheet: J1, Q1, R1, R2, U1
